Commit message: Add files via upload
updated as per our car

File: src/seav_bot/description/robot_core.xacro (robot description, xacro)
@@ -21,35 +21,74 @@
         <parent link="base_link"/>
         <child link="chassis"/>
-        <origin xyz="-0.1 0 0"/>
+        <origin xyz="0 0 0"/>
     </joint>
     <link name="chassis">
         <visual>
-            <origin xyz="0.15 0 0.075"/>
+            <origin xyz="0.55 0 0.20375"/>
             <geometry>
-                <box size="0.3 0.3 0.15"/>
+                <box size="1.10 0.52 0.1975"/>
+            </geometry>
+            <material name="white"/>
+        </visual>
+        <visual>
+            <origin xyz="0.0475 0 0.07875"/>
+            <geometry>
+                <box size="0.095 0.52 0.0525"/>
+            </geometry>
+            <material name="white"/>
+        </visual>
+        <visual>
+            <origin xyz="0.475 0 0.07875"/>
+            <geometry>
+                <box size="0.35 0.52 0.0525"/>
+            </geometry>
+            <material name="white"/>
+        </visual>
+        <visual>
+            <origin xyz="1.0025 0 0.07875"/>
+            <geometry>
+                <box size="0.195 0.52 0.0525"/>
             </geometry>
             <material name="white"/>
         </visual>
         <collision>
-            <origin xyz="0.15 0 0.075"/>
+            <origin xyz="0.55 0 0.20375"/>
             <geometry>
-                <box size="0.3 0.3 0.15"/>
+                <box size="1.10 0.52 0.1975"/>
             </geometry>
         </collision>
-        <xacro:inertial_box mass="0.5" x="0.3" y="0.3" z="0.15">
-            <origin xyz="0.15 0 0.075" rpy="0 0 0"/>
+        <collision>
+            <origin xyz="0.0475 0 0.07875"/>
+            <geometry>
+                <box size="0.095 0.52 0.0525"/>
+            </geometry>
+        </collision>
+        <collision>
+            <origin xyz="0.475 0 0.07875"/>
+            <geometry>
+                <box size="0.35 0.52 0.0525"/>
+            </geometry>
+        </collision>
+        <collision>
+            <origin xyz="1.0025 0 0.07875"/>
+            <geometry>
+                <box size="0.195 0.52 0.0525"/>
+            </geometry>
+        </collision>
+        <xacro:inertial_box mass="5.0" x="1.10" y="0.52" z="0.25">
+            <origin xyz="0.55 0 0.125" rpy="0 0 0"/>
         </xacro:inertial_box>
     </link>
-    <!-- LEFT WHEEL LINK -->
-    <joint name="left_wheel_joint" type="continuous">
-        <parent link="base_link"/>
-        <child link="left_wheel"/>
-        <origin xyz="0 0.175 0" rpy="-${pi/2} 0 0" />
+    <!-- REAR LEFT WHEEL LINK -->
+    <joint name="rear_left_wheel_joint" type="continuous">
+        <parent link="chassis"/>
+        <child link="rear_left_wheel"/>
+        <origin xyz="0.20 0.22 0" rpy="-${pi/2} 0 0" />
         <axis xyz="0 0 1"/>
     </joint>
-    <link name="left_wheel">
+    <link name="rear_left_wheel">
         <visual>
             <geometry>
-                <cylinder radius="0.05" length="0.04"/>
+                <cylinder radius="0.105" length="0.08"/>
             </geometry>
             <material name="blue"/>
@@ -57,22 +96,22 @@
         <collision>
             <geometry>
-                <cylinder radius="0.05" length="0.04"/>
+                <cylinder radius="0.105" length="0.08"/>
             </geometry>
         </collision>
-        <xacro:inertial_cylinder mass="0.1" length="0.04" radius="0.05">
+        <xacro:inertial_cylinder mass="1.0" length="0.08" radius="0.105">
             <origin xyz="0 0 0" rpy="0 0 0"/>
         </xacro:inertial_cylinder>
     </link>
-    <!-- RIGHT WHEEL LINK -->
-    <joint name="right_wheel_joint" type="continuous">
-        <parent link="base_link"/>
-        <child link="right_wheel"/>
-        <origin xyz="0 -0.175 0" rpy="${pi/2} 0 0" />
+    <!-- REAR RIGHT WHEEL LINK -->
+    <joint name="rear_right_wheel_joint" type="continuous">
+        <parent link="chassis"/>
+        <child link="rear_right_wheel"/>
+        <origin xyz="0.20 -0.22 0"  rpy="${pi/2} 0 0" />
         <axis xyz="0 0 -1"/>
     </joint>
-    <link name="right_wheel">
+    <link name="rear_right_wheel">
         <visual>
             <geometry>
-                <cylinder radius="0.05" length="0.04"/>
+                <cylinder radius="0.105" length="0.08"/>
             </geometry>
             <material name="blue"/>
@@ -80,32 +119,74 @@
         <collision>
             <geometry>
-                <cylinder radius="0.05" length="0.04"/>
+                <cylinder radius="0.105" length="0.08"/>
             </geometry>
         </collision>
-        <xacro:inertial_cylinder mass="0.1" length="0.04" radius="0.05">
+        <xacro:inertial_cylinder mass="1.0" length="0.08" radius="0.105">
             <origin xyz="0 0 0" rpy="0 0 0"/>
         </xacro:inertial_cylinder>
     </link>
-    <!-- CASTER WHEEL LINK -->
-    <joint name="caster_wheel_joint" type="fixed">
+    <!-- FRONT LEFT STEERING JOINT -->
+    <joint name="front_left_steering_joint" type="revolute">
         <parent link="chassis"/>
-        <child link="caster_wheel"/>
-        <origin xyz="0.24 0 0"/>
+        <child link="front_left_steering"/>
+        <origin xyz="0.78 0.22 0"/>
+        <axis xyz="0 0 1"/>
+        <limit lower="-0.75" upper="0.75" effort="1" velocity="1"/>
     </joint>
-    <link name="caster_wheel">
+    <link name="front_left_steering"/>
+    <!-- FRONT LEFT WHEEL ROLLING JOINT -->
+    <joint name="front_left_wheel_joint" type="continuous">
+        <parent link="front_left_steering"/>
+        <child link="front_left_wheel"/>
+        <origin xyz="0 0 0" rpy="-${pi/2} 0 0"/>
+        <axis xyz="0 0 1"/>
+    </joint>
+    <link name="front_left_wheel">
         <visual>
             <geometry>
-                <sphere radius="0.05"/>
+                <cylinder radius="0.105" length="0.08"/>
             </geometry>
-            <material name="black"/>
+            <material name="blue"/>
         </visual>
         <collision>
             <geometry>
-                <sphere radius="0.05"/>
+                <cylinder radius="0.105" length="0.08"/>
             </geometry>
         </collision>
-        <xacro:inertial_sphere mass="0.1" radius="0.05">
+        <xacro:inertial_cylinder mass="1.0" length="0.08" radius="0.105">
             <origin xyz="0 0 0" rpy="0 0 0"/>
-        </xacro:inertial_sphere>
+        </xacro:inertial_cylinder>
+    </link>
+    <!-- FRONT RIGHT STEERING JOINT -->
+    <joint name="front_right_steering_joint" type="revolute">
+        <parent link="chassis"/>
+        <child link="front_right_steering"/>
+        <origin xyz="0.78 -0.22 0"/>
+        <axis xyz="0 0 1"/>
+        <limit lower="-0.75" upper="0.75" effort="1" velocity="1"/>
+    </joint>
+    <link name="front_right_steering"/>
+    <!-- FRONT RIGHTWHEEL ROLLING JOINT -->
+    <joint name="front_right_wheel_joint" type="continuous">
+        <parent link="front_right_steering"/>
+        <child link="front_right_wheel"/>
+        <origin xyz="0 0 0" rpy="${pi/2} 0 0"/>
+        <axis xyz="0 0 1"/>
+    </joint>
+    <link name="front_right_wheel">
+        <visual>
+            <geometry>
+                <cylinder radius="0.105" length="0.08"/>
+            </geometry>
+            <material name="blue"/>
+        </visual>
+        <collision>
+            <geometry>
+                <cylinder radius="0.105" length="0.08"/>
+            </geometry>
+        </collision>
+        <xacro:inertial_cylinder mass="1.0" length="0.08" radius="0.105">
+            <origin xyz="0 0 0" rpy="0 0 0"/>
+        </xacro:inertial_cylinder>
     </link>
 </robot>

Commit message: launch file updated

File: src/seav_bot/description/robot_core.xacro (robot description, xacro)
@@ -134,5 +134,23 @@
         <limit lower="-0.75" upper="0.75" effort="1" velocity="1"/>
     </joint>
-    <link name="front_left_steering"/>
+    <link name="front_left_steering">
+    <visual>
+        <origin xyz="0 0 0"/>
+        <geometry>
+        <box size="0.001 0.001 0.001"/>
+        </geometry>
+        <material name="black"/>
+    </visual>
+    <collision>
+        <origin xyz="0 0 0"/>
+        <geometry>
+        <box size="0.001 0.001 0.001"/>
+        </geometry>
+    </collision>
+    <inertial>
+        <mass value="0.001"/>
+        <inertia ixx="1e-7" ixy="0.0" ixz="0.0" iyy="1e-7" iyz="0.0" izz="1e-7"/>
+    </inertial>
+    </link>
     <!-- FRONT LEFT WHEEL ROLLING JOINT -->
     <joint name="front_left_wheel_joint" type="continuous">
@@ -147,5 +165,5 @@
                 <cylinder radius="0.105" length="0.08"/>
             </geometry>
-            <material name="blue"/>
+            <material name="orange"/>
         </visual>
         <collision>
@@ -166,5 +184,23 @@
         <limit lower="-0.75" upper="0.75" effort="1" velocity="1"/>
     </joint>
-    <link name="front_right_steering"/>
+    <link name="front_right_steering">
+    <visual>
+        <origin xyz="0 0 0"/>
+        <geometry>
+        <box size="0.001 0.001 0.001"/>
+        </geometry>
+        <material name="black"/>
+    </visual>
+    <collision>
+        <origin xyz="0 0 0"/>
+        <geometry>
+        <box size="0.001 0.001 0.001"/>
+        </geometry>
+    </collision>
+    <inertial>
+        <mass value="0.001"/>
+        <inertia ixx="1e-7" ixy="0.0" ixz="0.0" iyy="1e-7" iyz="0.0" izz="1e-7"/>
+    </inertial>
+    </link>
     <!-- FRONT RIGHTWHEEL ROLLING JOINT -->
     <joint name="front_right_wheel_joint" type="continuous">
@@ -179,5 +215,5 @@
                 <cylinder radius="0.105" length="0.08"/>
             </geometry>
-            <material name="blue"/>
+            <material name="orange"/>
         </visual>
         <collision>
