Commit message: Add files via upload

File: src/seav_bot/description/robot.urdf.xacro (robot description, xacro)
@@ -1,4 +1,5 @@
 <?xml version="1.0"?>
 <robot xmlns:xacro="http://www.ros.org/wiki/xacro"  name="robot">
-    <xacro:include filename="robot_core.xacro" />
+    <xacro:include filename="robot_core.xacro"/>
+    <xacro:include filename="gazebo_control.xacro"/>
 </robot>

File: src/seav_bot/description/robot_core.xacro (robot description, xacro)
@@ -25,53 +25,14 @@
     <link name="chassis">
         <visual>
-            <origin xyz="0.55 0 0.20375"/>
-            <geometry>
-                <box size="1.10 0.52 0.1975"/>
+            <origin xyz="0.55 0 0.125"/>
+            <geometry>
+                <box size="1.10 0.36 0.25"/>
             </geometry>
             <material name="white"/>
         </visual>
-        <visual>
-            <origin xyz="0.0475 0 0.07875"/>
-            <geometry>
-                <box size="0.095 0.52 0.0525"/>
-            </geometry>
-            <material name="white"/>
-        </visual>
-        <visual>
-            <origin xyz="0.475 0 0.07875"/>
-            <geometry>
-                <box size="0.35 0.52 0.0525"/>
-            </geometry>
-            <material name="white"/>
-        </visual>
-        <visual>
-            <origin xyz="1.0025 0 0.07875"/>
-            <geometry>
-                <box size="0.195 0.52 0.0525"/>
-            </geometry>
-            <material name="white"/>
-        </visual>
-        <collision>
-            <origin xyz="0.55 0 0.20375"/>
-            <geometry>
-                <box size="1.10 0.52 0.1975"/>
-            </geometry>
-        </collision>
-        <collision>
-            <origin xyz="0.0475 0 0.07875"/>
-            <geometry>
-                <box size="0.095 0.52 0.0525"/>
-            </geometry>
-        </collision>
-        <collision>
-            <origin xyz="0.475 0 0.07875"/>
-            <geometry>
-                <box size="0.35 0.52 0.0525"/>
-            </geometry>
-        </collision>
-        <collision>
-            <origin xyz="1.0025 0 0.07875"/>
-            <geometry>
-                <box size="0.195 0.52 0.0525"/>
+        <collision>
+            <origin xyz="0.55 0 0.125"/>
+            <geometry>
+                <box size="1.10 0.36 0.25"/>
             </geometry>
         </collision>
@@ -80,4 +41,7 @@
         </xacro:inertial_box>
     </link>
+    <gazebo reference="chassis">
+        <material>Gazebo/White</material>
+    </gazebo>
     <!-- REAR LEFT WHEEL LINK -->
     <joint name="rear_left_wheel_joint" type="continuous">
@@ -103,4 +67,7 @@
         </xacro:inertial_cylinder>
     </link>
+    <gazebo reference="rear_left_wheel">
+        <material>Gazebo/Blue</material>
+    </gazebo>
     <!-- REAR RIGHT WHEEL LINK -->
     <joint name="rear_right_wheel_joint" type="continuous">
@@ -126,4 +93,7 @@
         </xacro:inertial_cylinder>
     </link>
+    <gazebo reference="rear_right_wheel">
+        <material>Gazebo/Blue</material>
+    </gazebo>
     <!-- FRONT LEFT STEERING JOINT -->
     <joint name="front_left_steering_joint" type="revolute">
@@ -176,4 +146,7 @@
         </xacro:inertial_cylinder>
     </link>
+    <gazebo reference="front_left_wheel">
+        <material>Gazebo/Orange</material>
+    </gazebo>
     <!-- FRONT RIGHT STEERING JOINT -->
     <joint name="front_right_steering_joint" type="revolute">
@@ -226,3 +199,12 @@
         </xacro:inertial_cylinder>
     </link>
+    <gazebo reference="front_right_wheel">
+        <material>Gazebo/Orange</material>
+    </gazebo>
+    <joint name="steering_wheel_joint" type="fixed">
+      <parent link="chassis"/>
+      <child link="steering_wheel_link"/>
+      <origin xyz="0 0 0"/>
+    </joint>
+    <link name="steering_wheel_link"/>
 </robot>
